File: encoder_daugtherboard.kicad_sch (KiCad schematic)
At the start: 12 parts, among them J10 Conn_01x02_Pin, J12 Conn_01x02_Pin, J14 Conn_01x02_Pin, J16 Conn_01x02_Pin, SW6 RotaryEncoder_Switch

Commit message: updating schematic
Parts:
- renumbered C50 to C601, C51 to C602, J10 to J601, J14 to J602, J12 to J603, J16 to J604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
