File: encoder_daugtherboard.kicad_sch (KiCad schematic)
At the start: 12 parts, among them J601 Conn_01x02_Pin, J602 Conn_01x02_Pin, J603 Conn_01x02_Pin, J604 Conn_01x02_Pin, SW601 RotaryEncoder_Switch

Commit message: voltage regulator circuit
routed the voltage regulator circuit following strongly suggested layout from the rp2350 hardware design doc, sized decoupling capacitors down
Parts:
- C601, C602: footprint Capacitor_SMD:C_1206_3216Metric -> Capacitor_SMD:C_0402_1005Metric
Changed lines of the file:
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@@
 			)
 		)
-		(property "Footprint" "Capacitor_SMD:C_1206_3216Metric"
+		(property "Footprint" "Capacitor_SMD:C_0402_1005Metric"
 			(at 82.55 38.1 0)
 			(hide yes)
@@
 			)
 		)
-		(property "Footprint" "Capacitor_SMD:C_1206_3216Metric"
+		(property "Footprint" "Capacitor_SMD:C_0402_1005Metric"
 			(at 44.45 38.1 0)
 			(hide yes)
