File: encoder_daugtherboard.kicad_sch (KiCad schematic)
At the start: 12 parts, among them J601 Conn_01x02_Pin, J602 Conn_01x02_Pin, J603 Conn_01x02_Pin, J604 Conn_01x02_Pin, SW601 RotaryEncoder_Switch

Commit message: minor adjustments
Parts:
- renumbered C601 to C701, C602 to C702, J601 to J701, J602 to J702, J603 to J703, J604 to J704, R601 to R701, R602 to R702, R603 to R703, R604 to R704, R605 to R705, SW601 to SW701
Changed lines of the file:
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@@
 	(generator "eeschema")
 	(generator_version "10.0")
-	(paper "User" 148.0000088 104.9999932)
+	(paper "User" 148 105)
 	(title_block
 		(title "Tome: Encoder Daughterboard")
@@
 		(in_pos_files yes)
 		(dnp no)
-		(property "Reference" "R602"
+		(property "Reference" "R702"
 			(at 60.706 25.146 0)
 			(show_name no)
@@
 				(path "/66975c75-2f34-465a-a19c-b694cfc16dd4/48ca1010-2b1c-4f07-a9f5-ed8eedc71556"
 					(reference "R?")
+					(unit 1)
+				)
+			)
+			(project "encoder_daugtherboard"
+				(path "/88308db8-3e55-4427-9961-760607475d1f"
+					(reference "R702")
 					(unit 1)
 				)
@@
 		(dnp no)
 		(fields_autoplaced yes)
-		(property "Reference" "#PWR0602"
+		(property "Reference" "#PWR0702"
 			(at 60.96 59.69 0)
 			(hide yes)
@@
 				(path "/66975c75-2f34-465a-a19c-b694cfc16dd4/48ca1010-2b1c-4f07-a9f5-ed8eedc71556"
 					(reference "#PWR0160")
+					(unit 1)
+				)
+			)
+			(project "encoder_daugtherboard"
+				(path "/88308db8-3e55-4427-9961-760607475d1f"
+					(reference "#PWR0702")
 					(unit 1)
 				)
@@
 		(in_pos_files yes)
 		(dnp no)
-		(property "Reference" "SW601"
+		(property "Reference" "SW701"
 			(at 69.85 41.656 0)
 			(show_name no)
@@
 				(path "/66975c75-2f34-465a-a19c-b694cfc16dd4/48ca1010-2b1c-4f07-a9f5-ed8eedc71556"
 					(reference "SW?")
+					(unit 1)
+				)
+			)
+			(project "encoder_daugtherboard"
+				(path "/88308db8-3e55-4427-9961-760607475d1f"
+					(reference "SW701")
 					(unit 1)
 				)
@@
 		(in_pos_files yes)
 		(dnp no)
-		(property "Reference" "R601"
+		(property "Reference" "R701"
 			(at 46.736 29.464 0)
 			(show_name no)
@@
 				(path "/66975c75-2f34-465a-a19c-b694cfc16dd4/48ca1010-2b1c-4f07-a9f5-ed8eedc71556"
 					(reference "R?")
+					(unit 1)
+				)
+			)
+			(project "encoder_daugtherboard"
+				(path "/88308db8-3e55-4427-9961-760607475d1f"
+					(reference "R701")
 					(unit 1)
 				)
@@
 		(dnp no)
 		(fields_autoplaced yes)
-		(property "Reference" "#PWR0604"
+		(property "Reference" "#PWR0704"
 			(at 82.55 53.34 0)
 			(hide yes)
@@
 				(path "/66975c75-2f34-465a-a19c-b694cfc16dd4/48ca1010-2b1c-4f07-a9f5-ed8eedc71556"
 					(reference "#PWR0158")
+					(unit 1)
+				)
+			)
+			(project "encoder_daugtherboard"
+				(path "/88308db8-3e55-4427-9961-760607475d1f"
+					(reference "#PWR0704")
 					(unit 1)
 				)
@@
 		(in_pos_files yes)
 		(dnp no)
-		(property "Reference" "R604"
+		(property "Reference" "R704"
 			(at 80.01 29.972 0)
 			(show_name no)
@@
 				(path "/66975c75-2f34-465a-a19c-b694cfc16dd4/48ca1010-2b1c-4f07-a9f5-ed8eedc71556"
 					(reference "R?")
+					(unit 1)
+				)
+			)
+			(project "encoder_daugtherboard"
+				(path "/88308db8-3e55-4427-9961-760607475d1f"
+					(reference "R704")
 					(unit 1)
 				)
@@
 		(dnp no)
 		(fields_autoplaced yes)
-		(property "Reference" "J604"
+		(property "Reference" "J704"
 			(at 112.395 35.56 0)
 			(show_name no)
@@
 				(path "/66975c75-2f34-465a-a19c-b694cfc16dd4/48ca1010-2b1c-4f07-a9f5-ed8eedc71556"
 					(reference "J?")
+					(unit 1)
+				)
+			)
+			(project "encoder_daugtherboard"
+				(path "/88308db8-3e55-4427-9961-760607475d1f"
+					(reference "J704")
 					(unit 1)
 				)
@@
 		(in_pos_files yes)
 		(dnp no)
-		(property "Reference" "R603"
+		(property "Reference" "R703"
 			(at 73.406 25.146 0)
 			(show_name no)
@@
 				(path "/66975c75-2f34-465a-a19c-b694cfc16dd4/48ca1010-2b1c-4f07-a9f5-ed8eedc71556"
 					(reference "R?")
+					(unit 1)
+				)
+			)
+			(project "encoder_daugtherboard"
+				(path "/88308db8-3e55-4427-9961-760607475d1f"
+					(reference "R703")
 					(unit 1)
 				)
@@
 		(dnp no)
 		(fields_autoplaced yes)
-		(property "Reference" "J603"
+		(property "Reference" "J703"
 			(at 112.395 15.24 0)
 			(show_name no)
@@
 				(path "/66975c75-2f34-465a-a19c-b694cfc16dd4/48ca1010-2b1c-4f07-a9f5-ed8eedc71556"
 					(reference "J?")
+					(unit 1)
+				)
+			)
+			(project "encoder_daugtherboard"
+				(path "/88308db8-3e55-4427-9961-760607475d1f"
+					(reference "J703")
 					(unit 1)
 				)
@@
 		(dnp no)
 		(fields_autoplaced yes)
-		(property "Reference" "#PWR0601"
+		(property "Reference" "#PWR0701"
 			(at 44.45 53.34 0)
 			(hide yes)
@@
 				(path "/66975c75-2f34-465a-a19c-b694cfc16dd4/48ca1010-2b1c-4f07-a9f5-ed8eedc71556"
 					(reference "#PWR0161")
+					(unit 1)
+				)
+			)
+			(project "encoder_daugtherboard"
+				(path "/88308db8-3e55-4427-9961-760607475d1f"
+					(reference "#PWR0701")
 					(unit 1)
 				)
@@
 		(dnp no)
 		(fields_autoplaced yes)
-		(property "Reference" "J601"
+		(property "Reference" "J701"
 			(at 22.225 15.24 0)
 			(show_name no)
@@
 				(path "/66975c75-2f34-465a-a19c-b694cfc16dd4/48ca1010-2b1c-4f07-a9f5-ed8eedc71556"
 					(reference "J?")
+					(unit 1)
+				)
+			)
+			(project "encoder_daugtherboard"
+				(path "/88308db8-3e55-4427-9961-760607475d1f"
+					(reference "J701")
 					(unit 1)
 				)
@@
 		(dnp no)
 		(fields_autoplaced yes)
-		(property "Reference" "#PWR0603"
+		(property "Reference" "#PWR0703"
 			(at 66.04 33.02 0)
 			(hide yes)
@@
 				(path "/66975c75-2f34-465a-a19c-b694cfc16dd4/48ca1010-2b1c-4f07-a9f5-ed8eedc71556"
 					(reference "#PWR0159")
+					(unit 1)
+				)
+			)
+			(project "encoder_daugtherboard"
+				(path "/88308db8-3e55-4427-9961-760607475d1f"
+					(reference "#PWR0703")
 					(unit 1)
 				)
@@
 		(dnp no)
 		(fields_autoplaced yes)
-		(property "Reference" "C602"
+		(property "Reference" "C702"
 			(at 85.09 36.8362 0)
 			(show_name no)
@@
 				(path "/66975c75-2f34-465a-a19c-b694cfc16dd4/48ca1010-2b1c-4f07-a9f5-ed8eedc71556"
 					(reference "C?")
+					(unit 1)
+				)
+			)
+			(project "encoder_daugtherboard"
+				(path "/88308db8-3e55-4427-9961-760607475d1f"
+					(reference "C702")
 					(unit 1)
 				)
@@
 		(in_pos_files yes)
 		(dnp no)
-		(property "Reference" "R605"
+		(property "Reference" "R705"
 			(at 105.156 45.466 0)
 			(show_name no)
@@
 				(path "/66975c75-2f34-465a-a19c-b694cfc16dd4/48ca1010-2b1c-4f07-a9f5-ed8eedc71556"
 					(reference "R?")
+					(unit 1)
+				)
+			)
+			(project "encoder_daugtherboard"
+				(path "/88308db8-3e55-4427-9961-760607475d1f"
+					(reference "R705")
 					(unit 1)
 				)
@@
 		(dnp no)
 		(fields_autoplaced yes)
-		(property "Reference" "J602"
+		(property "Reference" "J702"
 			(at 22.225 35.56 0)
 			(show_name no)
@@
 				(path "/66975c75-2f34-465a-a19c-b694cfc16dd4/48ca1010-2b1c-4f07-a9f5-ed8eedc71556"
 					(reference "J?")
+					(unit 1)
+				)
+			)
+			(project "encoder_daugtherboard"
+				(path "/88308db8-3e55-4427-9961-760607475d1f"
+					(reference "J702")
 					(unit 1)
 				)
@@
 		(dnp no)
 		(fields_autoplaced yes)
-		(property "Reference" "C601"
+		(property "Reference" "C701"
 			(at 46.99 36.8362 0)
 			(show_name no)
@@
 				)
 			)
-		)
-	)
+			(project "encoder_daugtherboard"
+				(path "/88308db8-3e55-4427-9961-760607475d1f"
+					(reference "C701")
+					(unit 1)
+				)
+			)
+		)
+	)
+	(sheet_instances
+		(path "/"
+			(page "1")
+		)
+	)
+	(embedded_fonts no)
 )

Commit message: spelling
Parts:
- renumbered C701 to C601, C702 to C602, J701 to J601, J702 to J602, J703 to J603, J704 to J604, R701 to R601, R702 to R602, R703 to R603, R704 to R604, R705 to R605, SW701 to SW601
Changed lines of the file:
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@@
 		(in_pos_files yes)
 		(dnp no)
-		(property "Reference" "R702"
+		(property "Reference" "R602"
 			(at 60.706 25.146 0)
 			(show_name no)
@@
 		(dnp no)
 		(fields_autoplaced yes)
-		(property "Reference" "#PWR0702"
+		(property "Reference" "#PWR0602"
 			(at 60.96 59.69 0)
 			(hide yes)
@@
 		(in_pos_files yes)
 		(dnp no)
-		(property "Reference" "SW701"
+		(property "Reference" "SW601"
 			(at 69.85 41.656 0)
 			(show_name no)
@@
 		(in_pos_files yes)
 		(dnp no)
-		(property "Reference" "R701"
+		(property "Reference" "R601"
 			(at 46.736 29.464 0)
 			(show_name no)
@@
 		(dnp no)
 		(fields_autoplaced yes)
-		(property "Reference" "#PWR0704"
+		(property "Reference" "#PWR0604"
 			(at 82.55 53.34 0)
 			(hide yes)
@@
 		(in_pos_files yes)
 		(dnp no)
-		(property "Reference" "R704"
+		(property "Reference" "R604"
 			(at 80.01 29.972 0)
 			(show_name no)
@@
 		(dnp no)
 		(fields_autoplaced yes)
-		(property "Reference" "J704"
+		(property "Reference" "J604"
 			(at 112.395 35.56 0)
 			(show_name no)
@@
 		(in_pos_files yes)
 		(dnp no)
-		(property "Reference" "R703"
+		(property "Reference" "R603"
 			(at 73.406 25.146 0)
 			(show_name no)
@@
 		(dnp no)
 		(fields_autoplaced yes)
-		(property "Reference" "J703"
+		(property "Reference" "J603"
 			(at 112.395 15.24 0)
 			(show_name no)
@@
 		(dnp no)
 		(fields_autoplaced yes)
-		(property "Reference" "#PWR0701"
+		(property "Reference" "#PWR0601"
 			(at 44.45 53.34 0)
 			(hide yes)
@@
 		(dnp no)
 		(fields_autoplaced yes)
-		(property "Reference" "J701"
+		(property "Reference" "J601"
 			(at 22.225 15.24 0)
 			(show_name no)
@@
 		(dnp no)
 		(fields_autoplaced yes)
-		(property "Reference" "#PWR0703"
+		(property "Reference" "#PWR0603"
 			(at 66.04 33.02 0)
 			(hide yes)
@@
 		(dnp no)
 		(fields_autoplaced yes)
-		(property "Reference" "C702"
+		(property "Reference" "C602"
 			(at 85.09 36.8362 0)
 			(show_name no)
@@
 		(in_pos_files yes)
 		(dnp no)
-		(property "Reference" "R705"
+		(property "Reference" "R605"
 			(at 105.156 45.466 0)
 			(show_name no)
@@
 		(dnp no)
 		(fields_autoplaced yes)
-		(property "Reference" "J702"
+		(property "Reference" "J602"
 			(at 22.225 35.56 0)
 			(show_name no)
@@
 		(dnp no)
 		(fields_autoplaced yes)
-		(property "Reference" "C701"
+		(property "Reference" "C601"
 			(at 46.99 36.8362 0)
 			(show_name no)
@@
 		)
 	)
-	(embedded_fonts no)
 )
