File: peripheral_mainboard.kicad_sch (KiCad schematic)
At the start: 34 parts, among them J5 AudioJack3, J9 FFC Connector, SW2 SW_SPST, SW3 SW_SPST, U5 TLV70033_SOT23-5, U6 PCM5102A, U7 PAM8908

Commit message: updating schematic
Parts:
- renumbered C18 to C301, C19 to C302, C38 to C303, C39 to C304, C35 to C305, C32 to C306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
