File: screen_daughterboard.kicad_sch (KiCad schematic)
At the start: 18 parts, among them J401 FPC Connector, Q401 Si1308EDL

Commit message: minor adjustments
Parts:
- renumbered C401 to C501, C402 to C502, C403 to C503, C404 to C504, C405 to C505, C406 to C506, C407 to C507, C408 to C508, C409 to C509, C410 to C510, D401 to D501, D402 to D502, D403 to D503, J401 to J501, L401 to L501, Q401 to Q501, R401 to R501, R402 to R502
Changed lines of the file:
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@@
 		(rev "1.0")
 		(company "rien+la_reine;")
-		(comment 1 "using GDEH0576T81 5.76” SPI display")
+		(comment 1 "using GDEH0576T81 5.76\" SPI display")
 		(comment 3 "SPDX-FileCopyrightText: 2026 Harsh Patel")
 		(comment 4 "SPDX-License-Identifier: CERN-OHL-S-2.0")
@@
 		(in_pos_files yes)
 		(dnp no)
-		(property "Reference" "D401"
+		(property "Reference" "D501"
 			(at 144.78 73.406 0)
 			(show_name no)
@@
 				)
 			)
+			(project "screen_daughterboard"
+				(path "/6f7248e0-d3a6-4d93-8705-a70cd5c1da40"
+					(reference "D501")
+					(unit 1)
+				)
+			)
 		)
 	)
@@
 		(dnp no)
 		(fields_autoplaced yes)
-		(property "Reference" "R401"
+		(property "Reference" "R501"
 			(at 130.81 54.6099 0)
 			(show_name no)
@@
 				)
 			)
+			(project "screen_daughterboard"
+				(path "/6f7248e0-d3a6-4d93-8705-a70cd5c1da40"
+					(reference "R501")
+					(unit 1)
+				)
+			)
 		)
 	)
@@
 		(dnp no)
 		(fields_autoplaced yes)
-		(property "Reference" "C407"
+		(property "Reference" "C507"
 			(at 114.3 40.6335 0)
 			(show_name no)
@@
 				)
 			)
+			(project "screen_daughterboard"
+				(path "/6f7248e0-d3a6-4d93-8705-a70cd5c1da40"
+					(reference "C507")
+					(unit 1)
+				)
+			)
 		)
 	)
@@
 		(dnp no)
 		(fields_autoplaced yes)
-		(property "Reference" "J401"
+		(property "Reference" "J501"
 			(at 64.77 73.6599 0)
 			(show_name no)
@@
 				)
 			)
+			(project "screen_daughterboard"
+				(path "/6f7248e0-d3a6-4d93-8705-a70cd5c1da40"
+					(reference "J501")
+					(unit 1)
+				)
+			)
 		)
 	)
@@
 		(dnp no)
 		(fields_autoplaced yes)
-		(property "Reference" "#PWR0404"
+		(property "Reference" "#PWR0504"
 			(at 143.51 90.17 0)
 			(hide yes)
@@
 				)
 			)
+			(project "screen_daughterboard"
+				(path "/6f7248e0-d3a6-4d93-8705-a70cd5c1da40"
+					(reference "#PWR0504")
+					(unit 1)
+				)
+			)
 		)
 	)
@@
 		(dnp no)
 		(fields_autoplaced yes)
-		(property "Reference" "#PWR0402"
+		(property "Reference" "#PWR0502"
 			(at 111.76 53.34 0)
 			(hide yes)
@@
 				)
 			)
+			(project "screen_daughterboard"
+				(path "/6f7248e0-d3a6-4d93-8705-a70cd5c1da40"
+					(reference "#PWR0502")
+					(unit 1)
+				)
+			)
 		)
 	)
@@
 		(dnp no)
 		(fields_autoplaced yes)
-		(property "Reference" "#PWR0405"
+		(property "Reference" "#PWR0505"
 			(at 153.67 92.71 0)
 			(hide yes)
@@
 				)
 			)
+			(project "screen_daughterboard"
+				(path "/6f7248e0-d3a6-4d93-8705-a70cd5c1da40"
+					(reference "#PWR0505")
+					(unit 1)
+				)
+			)
 		)
 	)
@@
 		(dnp no)
 		(fields_autoplaced yes)
-		(property "Reference" "C403"
+		(property "Reference" "C503"
 			(at 33.0263 92.71 90)
 			(show_name no)
@@
 				)
 			)
+			(project "screen_daughterboard"
+				(path "/6f7248e0-d3a6-4d93-8705-a70cd5c1da40"
+					(reference "C503")
+					(unit 1)
+				)
+			)
 		)
 	)
@@
 		(dnp no)
 		(fields_autoplaced yes)
-		(property "Reference" "C406"
+		(property "Reference" "C506"
 			(at 40.6463 97.79 90)
 			(show_name no)
@@
 				)
 			)
+			(project "screen_daughterboard"
+				(path "/6f7248e0-d3a6-4d93-8705-a70cd5c1da40"
+					(reference "C506")
+					(unit 1)
+				)
+			)
 		)
 	)
@@
 		(dnp no)
 		(fields_autoplaced yes)
-		(property "Reference" "L401"
+		(property "Reference" "L501"
 			(at 116.84 33.02 90)
 			(show_name no)
@@
 				)
 			)
+			(project "screen_daughterboard"
+				(path "/6f7248e0-d3a6-4d93-8705-a70cd5c1da40"
+					(reference "L501")
+					(unit 1)
+				)
+			)
 		)
 	)
@@
 		(dnp no)
 		(fields_autoplaced yes)
-		(property "Reference" "C405"
+		(property "Reference" "C505"
 			(at 40.6463 87.63 90)
 			(show_name no)
@@
 				)
 			)
+			(project "screen_daughterboard"
+				(path "/6f7248e0-d3a6-4d93-8705-a70cd5c1da40"
+					(reference "C505")
+					(unit 1)
+				)
+			)
 		)
 	)
@@
 		(dnp no)
 		(fields_autoplaced yes)
-		(property "Reference" "R402"
+		(property "Reference" "R502"
 			(at 139.7 54.6099 0)
 			(show_name no)
@@
 				)
 			)
+			(project "screen_daughterboard"
+				(path "/6f7248e0-d3a6-4d93-8705-a70cd5c1da40"
+					(reference "R502")
+					(unit 1)
+				)
+			)
 		)
 	)
@@
 		(in_pos_files yes)
 		(dnp no)
-		(property "Reference" "D403"
+		(property "Reference" "D503"
 			(at 174.752 83.312 0)
 			(show_name no)
@@
 				)
 			)
+			(project "screen_daughterboard"
+				(path "/6f7248e0-d3a6-4d93-8705-a70cd5c1da40"
+					(reference "D503")
+					(unit 1)
+				)
+			)
 		)
 	)
@@
 		(dnp no)
 		(fields_autoplaced yes)
-		(property "Reference" "Q401"
+		(property "Reference" "Q501"
 			(at 140.97 44.4499 0)
 			(show_name no)
@@
 				)
 			)
+			(project "screen_daughterboard"
+				(path "/6f7248e0-d3a6-4d93-8705-a70cd5c1da40"
+					(reference "Q501")
+					(unit 1)
+				)
+			)
 		)
 	)
@@
 		(dnp no)
 		(fields_autoplaced yes)
-		(property "Reference" "C408"
+		(property "Reference" "C508"
 			(at 146.05 77.4635 0)
 			(show_name no)
@@
 				)
 			)
+			(project "screen_daughterboard"
+				(path "/6f7248e0-d3a6-4d93-8705-a70cd5c1da40"
+					(reference "C508")
+					(unit 1)
+				)
+			)
 		)
 	)
@@
 		(dnp no)
 		(fields_autoplaced yes)
-		(property "Reference" "C409"
+		(property "Reference" "C509"
 			(at 156.21 67.3035 0)
 			(show_name no)
@@
 				)
 			)
+			(project "screen_daughterboard"
+				(path "/6f7248e0-d3a6-4d93-8705-a70cd5c1da40"
+					(reference "C509")
+					(unit 1)
+				)
+			)
 		)
 	)
@@
 		(dnp no)
 		(fields_autoplaced yes)
-		(property "Reference" "#PWR0403"
+		(property "Reference" "#PWR0503"
 			(at 137.16 67.31 0)
 			(hide yes)
@@
 				)
 			)
+			(project "screen_daughterboard"
+				(path "/6f7248e0-d3a6-4d93-8705-a70cd5c1da40"
+					(reference "#PWR0503")
+					(unit 1)
+				)
+			)
 		)
 	)
@@
 		(in_pos_files yes)
 		(dnp no)
-		(property "Reference" "D402"
+		(property "Reference" "D502"
 			(at 154.94 84.836 0)
 			(show_name no)
@@
 				)
 			)
+			(project "screen_daughterboard"
+				(path "/6f7248e0-d3a6-4d93-8705-a70cd5c1da40"
+					(reference "D502")
+					(unit 1)
+				)
+			)
 		)
 	)
@@
 		(dnp no)
 		(fields_autoplaced yes)
-		(property "Reference" "C410"
+		(property "Reference" "C510"
 			(at 175.26 87.6235 0)
 			(show_name no)
@@
 				)
 			)
+			(project "screen_daughterboard"
+				(path "/6f7248e0-d3a6-4d93-8705-a70cd5c1da40"
+					(reference "C510")
+					(unit 1)
+				)
+			)
 		)
 	)
@@
 		(dnp no)
 		(fields_autoplaced yes)
-		(property "Reference" "C402"
+		(property "Reference" "C502"
 			(at 33.0263 82.55 90)
 			(show_name no)
@@
 				)
 			)
+			(project "screen_daughterboard"
+				(path "/6f7248e0-d3a6-4d93-8705-a70cd5c1da40"
+					(reference "C502")
+					(unit 1)
+				)
+			)
 		)
 	)
@@
 		(dnp no)
 		(fields_autoplaced yes)
-		(property "Reference" "#PWR0406"
+		(property "Reference" "#PWR0506"
 			(at 172.72 100.33 0)
 			(hide yes)
@@
 				)
 			)
+			(project "screen_daughterboard"
+				(path "/6f7248e0-d3a6-4d93-8705-a70cd5c1da40"
+					(reference "#PWR0506")
+					(unit 1)
+				)
+			)
 		)
 	)
@@
 		(dnp no)
 		(fields_autoplaced yes)
-		(property "Reference" "C404"
+		(property "Reference" "C504"
 			(at 34.2963 49.53 90)
 			(show_name no)
@@
 				)
 			)
+			(project "screen_daughterboard"
+				(path "/6f7248e0-d3a6-4d93-8705-a70cd5c1da40"
+					(reference "C504")
+					(unit 1)
+				)
+			)
 		)
 	)
@@
 		(dnp no)
 		(fields_autoplaced yes)
-		(property "Reference" "#PWR0401"
+		(property "Reference" "#PWR0501"
 			(at 22.86 113.03 0)
 			(hide yes)
@@
 				)
 			)
+			(project "screen_daughterboard"
+				(path "/6f7248e0-d3a6-4d93-8705-a70cd5c1da40"
+					(reference "#PWR0501")
+					(unit 1)
+				)
+			)
 		)
 	)
@@
 		(dnp no)
 		(fields_autoplaced yes)
-		(property "Reference" "C401"
+		(property "Reference" "C501"
 			(at 29.2163 74.93 90)
 			(show_name no)
@@
 				)
 			)
+			(project "screen_daughterboard"
+				(path "/6f7248e0-d3a6-4d93-8705-a70cd5c1da40"
+					(reference "C501")
+					(unit 1)
+				)
+			)
+		)
+	)
+	(sheet_instances
+		(path "/"
+			(page "1")
 		)
 	)
+	(embedded_fonts no)
 )

Commit message: spelling
Parts:
- renumbered C501 to C401, C502 to C402, C503 to C403, C504 to C404, C505 to C405, C506 to C406, C507 to C407, C508 to C408, C509 to C409, C510 to C410, D501 to D401, D502 to D402, D503 to D403, J501 to J401, L501 to L401, Q501 to Q401, R501 to R401, R502 to R402
Changed lines of the file:
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@@
 		(in_pos_files yes)
 		(dnp no)
-		(property "Reference" "D501"
+		(property "Reference" "D401"
 			(at 144.78 73.406 0)
 			(show_name no)
@@
 		(dnp no)
 		(fields_autoplaced yes)
-		(property "Reference" "R501"
+		(property "Reference" "R401"
 			(at 130.81 54.6099 0)
 			(show_name no)
@@
 		(dnp no)
 		(fields_autoplaced yes)
-		(property "Reference" "C507"
+		(property "Reference" "C407"
 			(at 114.3 40.6335 0)
 			(show_name no)
@@
 		(dnp no)
 		(fields_autoplaced yes)
-		(property "Reference" "J501"
+		(property "Reference" "J401"
 			(at 64.77 73.6599 0)
 			(show_name no)
@@
 		(dnp no)
 		(fields_autoplaced yes)
-		(property "Reference" "#PWR0504"
+		(property "Reference" "#PWR0404"
 			(at 143.51 90.17 0)
 			(hide yes)
@@
 		(dnp no)
 		(fields_autoplaced yes)
-		(property "Reference" "#PWR0502"
+		(property "Reference" "#PWR0402"
 			(at 111.76 53.34 0)
 			(hide yes)
@@
 		(dnp no)
 		(fields_autoplaced yes)
-		(property "Reference" "#PWR0505"
+		(property "Reference" "#PWR0405"
 			(at 153.67 92.71 0)
 			(hide yes)
@@
 		(dnp no)
 		(fields_autoplaced yes)
-		(property "Reference" "C503"
+		(property "Reference" "C403"
 			(at 33.0263 92.71 90)
 			(show_name no)
@@
 		(dnp no)
 		(fields_autoplaced yes)
-		(property "Reference" "C506"
+		(property "Reference" "C406"
 			(at 40.6463 97.79 90)
 			(show_name no)
@@
 		(dnp no)
 		(fields_autoplaced yes)
-		(property "Reference" "L501"
+		(property "Reference" "L401"
 			(at 116.84 33.02 90)
 			(show_name no)
@@
 		(dnp no)
 		(fields_autoplaced yes)
-		(property "Reference" "C505"
+		(property "Reference" "C405"
 			(at 40.6463 87.63 90)
 			(show_name no)
@@
 		(dnp no)
 		(fields_autoplaced yes)
-		(property "Reference" "R502"
+		(property "Reference" "R402"
 			(at 139.7 54.6099 0)
 			(show_name no)
@@
 		(in_pos_files yes)
 		(dnp no)
-		(property "Reference" "D503"
+		(property "Reference" "D403"
 			(at 174.752 83.312 0)
 			(show_name no)
@@
 		(dnp no)
 		(fields_autoplaced yes)
-		(property "Reference" "Q501"
+		(property "Reference" "Q401"
 			(at 140.97 44.4499 0)
 			(show_name no)
@@
 		(dnp no)
 		(fields_autoplaced yes)
-		(property "Reference" "C508"
+		(property "Reference" "C408"
 			(at 146.05 77.4635 0)
 			(show_name no)
@@
 		(dnp no)
 		(fields_autoplaced yes)
-		(property "Reference" "C509"
+		(property "Reference" "C409"
 			(at 156.21 67.3035 0)
 			(show_name no)
@@
 		(dnp no)
 		(fields_autoplaced yes)
-		(property "Reference" "#PWR0503"
+		(property "Reference" "#PWR0403"
 			(at 137.16 67.31 0)
 			(hide yes)
@@
 		(in_pos_files yes)
 		(dnp no)
-		(property "Reference" "D502"
+		(property "Reference" "D402"
 			(at 154.94 84.836 0)
 			(show_name no)
@@
 		(dnp no)
 		(fields_autoplaced yes)
-		(property "Reference" "C510"
+		(property "Reference" "C410"
 			(at 175.26 87.6235 0)
 			(show_name no)
@@
 		(dnp no)
 		(fields_autoplaced yes)
-		(property "Reference" "C502"
+		(property "Reference" "C402"
 			(at 33.0263 82.55 90)
 			(show_name no)
@@
 		(dnp no)
 		(fields_autoplaced yes)
-		(property "Reference" "#PWR0506"
+		(property "Reference" "#PWR0406"
 			(at 172.72 100.33 0)
 			(hide yes)
@@
 		(dnp no)
 		(fields_autoplaced yes)
-		(property "Reference" "C504"
+		(property "Reference" "C404"
 			(at 34.2963 49.53 90)
 			(show_name no)
@@
 		(dnp no)
 		(fields_autoplaced yes)
-		(property "Reference" "#PWR0501"
+		(property "Reference" "#PWR0401"
 			(at 22.86 113.03 0)
 			(hide yes)
@@
 		(dnp no)
 		(fields_autoplaced yes)
-		(property "Reference" "C501"
+		(property "Reference" "C401"
 			(at 29.2163 74.93 90)
 			(show_name no)
@@
 		)
 	)
-	(embedded_fonts no)
 )
